File: LABN1_SRA/kicad/LABN1_SRA/LABN1_SRA.kicad_pcb (KiCad board)
At the start: 2 copper layers, 130.8 x 70.5 mm, 40 parts, among them J1 Conn_01x03, J10 Conn_01x03, J2 Conn_01x02, J3 Conn_01x01, J4 Conn_01x02, J5 Conn_01x01, J6 Conn_01x02, J7 Conn_01x01, J8 Conn_01x01, J9 Conn_01x01, U1 LM324, U2 LM324

Commit message: updated kicad
Parts:
- R19: footprint Resistor_THT:R_Axial_DIN0309_L9.0mm_D3.2mm_P15.24mm_Horizontal -> Potentiometer_THT:Potentiometer_ACP_CA9-H3,8_Horizontal
- moved R19 4.00 mm to (132.5, 87.8), turned to 90 degrees

Commit message: informes actualizados
Parts:
- added J11: Conn_01x01, Connector_PinHeader_2.54mm:PinHeader_1x01_P2.54mm_Vertical, F.Cu at (145.0, 85.3)
Connections:
- R17 pad 1: GND -> Vref_D
Routing:
- net GND: track 14.6 -> 5.08 mm
- net Vref_D: track 0.00 -> 4.49 mm
Other:
- board text added: "GND"
- board text added: "V1_A|V2_A"
- board text added: "V1_B"
- board text added: "VCC|NC|VEE"
- board text added: "Vi_D"
- board text added: "Vin_C"
- board text added: "Vo1_A|Vo2_A"
- board text added: "Vo1_C|Vo2_C"
- board text added: "Vo_B"
- board text added: "Vo_D"
- board text added: "Vref_D"
