File: LABN1_SRA/kicad/LABN1_SRA/LABN1_SRA.kicad_sch (KiCad schematic)
At the start: 32 parts, among them J1 Conn_01x03, J10 Conn_01x03, J2 Conn_01x02, J3 Conn_01x01, J4 Conn_01x02, J5 Conn_01x01, J6 Conn_01x02, J7 Conn_01x01, J8 Conn_01x01, J9 Conn_01x01, U1 LM324, U2 LM324

Commit message: updated kicad
Parts:
- R19: footprint Resistor_THT:R_Axial_DIN0309_L9.0mm_D3.2mm_P15.24mm_Horizontal -> Potentiometer_THT:Potentiometer_ACP_CA9-H3,8_Horizontal
Changed lines of the file:
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@@
 			)
 		)
-		(property "Footprint" "Resistor_THT:R_Axial_DIN0309_L9.0mm_D3.2mm_P15.24mm_Horizontal"
+		(property "Footprint" "Potentiometer_THT:Potentiometer_ACP_CA9-H3,8_Horizontal"
 			(at 216.662 63.5 90)
 			(effects

Commit message: informes actualizados
Parts:
- added J11: Conn_01x01, Connector_PinHeader_2.54mm:PinHeader_1x01_P2.54mm_Vertical, symbol Connector_Generic:Conn_01x01
Connections:
- net GND: no longer R17.1
- new net Vref_D: J11.1 (Pin_1), R17.1
Changed lines of the file:
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@@
 	(wire
 		(pts
-			(xy 228.6 128.27) (xy 222.25 128.27)
+			(xy 222.25 128.27) (xy 228.6 128.27)
 		)
 		(stroke
@@
 	(wire
 		(pts
+			(xy 228.6 140.97) (xy 226.06 140.97)
+		)
+		(stroke
+			(width 0)
+			(type default)
+		)
+	)
+	(wire
+		(pts
 			(xy 128.27 60.96) (xy 130.81 60.96)
 		)
@@
 	(wire
 		(pts
-			(xy 85.09 162.56) (xy 83.82 162.56)
+			(xy 228.6 138.43) (xy 228.6 140.97)
 		)
 		(stroke
@@
 	(wire
 		(pts
-			(xy 214.63 54.61) (xy 218.44 54.61)
+			(xy 85.09 162.56) (xy 83.82 162.56)
 		)
 		(stroke
@@
 	(wire
 		(pts
-			(xy 228.6 138.43) (xy 228.6 139.7)
+			(xy 214.63 54.61) (xy 218.44 54.61)
 		)
 		(stroke
@@
 	(wire
 		(pts
+			(xy 149.86 168.91) (xy 152.4 168.91)
+		)
+		(stroke
+			(width 0)
+			(type default)
+		)
+	)
+	(wire
+		(pts
 			(xy 67.31 109.22) (xy 72.39 109.22)
 		)
@@
 		)
 	)
+	(global_label "Vref_D"
+		(shape input)
+		(at 226.06 140.97 180)
+		(fields_autoplaced yes)
+		(effects
+			(font
+				(size 1.27 1.27)
+			)
+			(justify right)
+		)
+		(property "Intersheetrefs" "${INTERSHEET_REFS}"
+			(at 217.1481 140.97 0)
+			(effects
+				(font
+					(size 1.27 1.27)
+				)
+				(justify right)
+				(hide yes)
+			)
+		)
+	)
 	(global_label "Vo2_A"
 		(shape output)
@@
 		)
 	)
+	(global_label "Vref_D"
+		(shape input)
+		(at 149.86 168.91 180)
+		(fields_autoplaced yes)
+		(effects
+			(font
+				(size 1.27 1.27)
+			)
+			(justify right)
+		)
+		(property "Intersheetrefs" "${INTERSHEET_REFS}"
+			(at 140.9481 168.91 0)
+			(effects
+				(font
+					(size 1.27 1.27)
+				)
+				(justify right)
+				(hide yes)
+			)
+		)
+	)
 	(global_label "V1_B"
 		(shape input)
@@
 	)
 	(symbol
+		(lib_id "Connector_Generic:Conn_01x01")
+		(at 157.48 168.91 0)
+		(unit 1)
+		(exclude_from_sim no)
+		(in_bom yes)
+		(on_board yes)
+		(dnp no)
+		(fields_autoplaced yes)
+		(property "Reference" "J11"
+			(at 160.02 167.6399 0)
+			(effects
+				(font
+					(size 1.27 1.27)
+				)
+				(justify left)
+			)
+		)
+		(property "Value" "Conn_01x01"
+			(at 160.02 170.1799 0)
+			(effects
+				(font
+					(size 1.27 1.27)
+				)
+				(justify left)
+			)
+		)
+		(property "Footprint" "Connector_PinHeader_2.54mm:PinHeader_1x01_P2.54mm_Vertical"
+			(at 157.48 168.91 0)
+			(effects
+				(font
+					(size 1.27 1.27)
+				)
+				(hide yes)
+			)
+		)
+		(property "Datasheet" "~"
+			(at 157.48 168.91 0)
+			(effects
+				(font
+					(size 1.27 1.27)
+				)
+				(hide yes)
+			)
+		)
+		(property "Description" "Generic connector, single row, 01x01, script generated (kicad-library-utils/schlib/autogen/connector/)"
+			(at 157.48 168.91 0)
+			(effects
+				(font
+					(size 1.27 1.27)
+				)
+				(hide yes)
+			)
+		)
+		(pin "1"
+		)
+		(instances
+			(project "LABN1_SRA"
+				(path "/5dad8d9f-335b-4703-a910-df4a2d6de689"
+					(reference "J11")
+					(unit 1)
+				)
+			)
+		)
+	)
+	(symbol
 		(lib_id "Diode:1N4148")
 		(at 96.52 104.14 90)
@@
 					(unit 1)
 				)
-			)
-		)
-	)
-	(symbol
-		(lib_id "power:GND")
-		(at 228.6 139.7 0)
-		(unit 1)
-		(exclude_from_sim no)
-		(in_bom yes)
-		(on_board yes)
-		(dnp no)
-		(fields_autoplaced yes)
-		(property "Reference" "#PWR05"
-			(at 228.6 146.05 0)
-			(effects
-				(font
-					(size 1.27 1.27)
-				)
-				(hide yes)
-			)
-		)
-		(property "Value" "GND"
-			(at 228.6 144.78 0)
-			(effects
-				(font
-					(size 1.27 1.27)
-				)
-			)
-		)
-		(property "Footprint" ""
-			(at 228.6 139.7 0)
-			(effects
-				(font
-					(size 1.27 1.27)
-				)
-				(hide yes)
-			)
-		)
-		(property "Datasheet" ""
-			(at 228.6 139.7 0)
-			(effects
-				(font
-					(size 1.27 1.27)
-				)
-				(hide yes)
-			)
-		)
-		(property "Description" "Power symbol creates a global label with name \"GND\" , ground"
-			(at 228.6 139.7 0)
-			(effects
-				(font
-					(size 1.27 1.27)
-				)
-				(hide yes)
-			)
-		)
-		(pin "1"
-		)
-		(instances
-			(project ""
-				(path "/5dad8d9f-335b-4703-a910-df4a2d6de689"
-					(reference "#PWR05")
-					(unit 1)
-				)
