File: LABN2_SRA/kicad/LABN2_SRA/LABN2_SRA.kicad_pcb (KiCad board)
At the start: 2 copper layers, 59.7 x 68.2 mm, 13 parts, among them J1 Conn_01x03, J2 Conn_01x03, J3 Conn_01x03, J4 Conn_01x03, U1 LM324

Commit message: actualizados archivos kicad a la ultima version
Parts:
- moved J3 42.8 mm to (145.8, 65.1)
- moved J4 42.8 mm to (160.4, 65.0)
- moved R1 42.8 mm to (140.9, 76.5)
- moved R2 42.8 mm to (140.9, 83.1)
- moved R6 42.8 mm to (153.9, 92.4)
- moved R7 42.8 mm to (143.7, 107.7)
- moved R8 42.8 mm to (147.2, 107.7)
- moved J1 42.8 mm to (162.3, 115.9)
- moved J2 42.8 mm to (141.9, 89.4)
- moved U1 42.8 mm to (147.3, 70.6)
- moved R3 42.8 mm to (125.7, 70.1)
- moved R4 42.8 mm to (165.7, 107.6)
- moved R5 42.8 mm to (159.7, 107.6)
